File: e.kicad_pcb (KiCad board)
At the start: 2 copper layers, 78 x 58.5 mm, 10 parts, among them SW1 usr, SW2 rst, U1 Display_ST7789, U2 MAX98357A

Commit message: almost done i hope
Parts:
- removed R3: 10K, Resistor_SMD:R_1206_3216Metric
Connections:
- BT1 pad 1: Net-(BT1-+) -> +3V0
Routing:
- net +3V0: track 115.6 -> 167.5 mm
- net Net-(BT1-+): track 47.3 -> 0.00 mm, vias 1 -> 0
Changed lines of the file:
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@@
 		)
 	)
-	(footprint "Resistor_SMD:R_1206_3216Metric"
-		(layer "F.Cu")
-		(at 142.15 110.65)
-		(descr "Resistor SMD 1206 (3216 Metric), square (rectangular) end terminal, IPC-7351 nominal, (Body size source: IPC-SM-782 page 72, https://www.pcb-3d.com/wordpress/wp-content/uploads/ipc-sm-782a_amendment_1_and_2.pdf)")
-		(tags "resistor")
-		(property "Reference" "R3"
-			(at 0 -1.83 0)
-			(layer "F.SilkS")
-			(effects
-				(font
-					(size 1 1)
-					(thickness 0.15)
-				)
-			)
-		)
-		(property "Value" "10K"
-			(at 0 1.83 0)
-			(layer "F.Fab")
-			(effects
-				(font
-					(size 1 1)
-					(thickness 0.15)
-				)
-			)
-		)
-		(property "Datasheet" ""
-			(at 0 0 0)
-			(layer "F.Fab")
-			(hide yes)
-			(effects
-				(font
-					(size 1.27 1.27)
-				)
-			)
-		)
-		(property "Description" "Resistor, small US symbol"
-			(at 0 0 0)
-			(layer "F.Fab")
-			(hide yes)
-			(effects
-				(font
-					(size 1.27 1.27)
-				)
-			)
-		)
-		(property ki_fp_filters "R_*")
-		(sheetname "/")
-		(sheetfile "e.kicad_sch")
-		(units
-			(unit
-				(name "A")
-				(pins "1" "2")
-			)
-		)
-		(attr smd)
-		(duplicate_pad_numbers_are_jumpers no)
-		(fp_line
-			(start -0.727064 -0.91)
-			(end 0.727064 -0.91)
-			(stroke
-				(width 0.12)
-				(type solid)
-			)
-			(layer "F.SilkS")
-		)
-		(fp_line
-			(start -0.727064 0.91)
-			(end 0.727064 0.91)
-			(stroke
-				(width 0.12)
-				(type solid)
-			)
-			(layer "F.SilkS")
-		)
-		(fp_rect
-			(start -2.28 -1.13)
-			(end 2.28 1.13)
-			(stroke
-				(width 0.05)
-				(type solid)
-			)
-			(fill no)
-			(layer "F.CrtYd")
-		)
-		(fp_rect
-			(start -1.6 -0.8)
-			(end 1.6 0.8)
-			(stroke
-				(width 0.1)
-				(type solid)
-			)
-			(fill no)
-			(layer "F.Fab")
-		)
-		(fp_text user "${REFERENCE}"
-			(at 0 0 0)
-			(layer "F.Fab")
-			(effects
-				(font
-					(size 0.8 0.8)
-					(thickness 0.12)
-				)
-			)
-		)
-		(pad "1" smd roundrect
-			(at -1.4625 0)
-			(size 1.125 1.75)
-			(layers "F.Cu" "F.Mask" "F.Paste")
-			(roundrect_rratio 0.222222)
-			(net "+3V0")
-			(pintype "passive")
-		)
-		(pad "2" smd roundrect
-			(at 1.4625 0)
-			(size 1.125 1.75)
-			(layers "F.Cu" "F.Mask" "F.Paste")
-			(roundrect_rratio 0.222222)
-			(net "Net-(BT1-+)")
-			(pintype "passive")
-		)
-		(embedded_fonts no)
-		(model "${KICAD10_3DMODEL_DIR}/Resistor_SMD.3dshapes/R_1206_3216Metric.step"
-			(offset
-				(xyz 0 0 0)
-			)
-			(scale
-				(xyz 1 1 1)
-			)
-			(rotate
-				(xyz 0 0 0)
-			)
-		)
-	)
 	(footprint "Button_Switch_THT:SW_Slide_SPDT_Straight_CK_OS102011MS2Q"
 		(layer "F.Cu")
@@
 			(size 6 5.5)
 			(layers "B.Cu" "B.Mask" "B.Paste")
-			(net "Net-(BT1-+)")
+			(net "+3V0")
 			(pinfunction "+_1")
 			(pintype "passive")
@@
 			(size 6 5.5)
 			(layers "B.Cu" "B.Mask" "B.Paste")
-			(net "Net-(BT1-+)")
+			(net "+3V0")
 			(pinfunction "+_1")
 			(pintype "passive")
@@
 	)
 	(segment
+		(start 141.15 103.95)
+		(end 141.15 109.65)
+		(width 0.2)
+		(layer "B.Cu")
+		(net "+3V0")
+	)
+	(segment
 		(start 183.15 78.15)
 		(end 183.15 78.65)
@@
 	)
 	(segment
+		(start 130.85 93.65)
+		(end 130.85 83.65)
+		(width 0.2)
+		(layer "B.Cu")
+		(net "+3V0")
+	)
+	(segment
+		(start 130.85 83.65)
+		(end 141.15 73.35)
+		(width 0.2)
+		(layer "B.Cu")
+		(net "+3V0")
+	)
+	(segment
 		(start 154.15 122.65)
 		(end 146.15 114.65)
@@
 	)
 	(segment
-		(start 153.85 75.21)
-		(end 156.85 72.21)
+		(start 141.15 103.95)
+		(end 130.85 93.65)
+		(width 0.2)
+		(layer "B.Cu")
+		(net "+3V0")
+	)
+	(segment
+		(start 141.15 109.65)
+		(end 146.15 114.65)
+		(width 0.2)
+		(layer "B.Cu")
+		(net "+3V0")
+	)
+	(segment
+		(start 147.15 68.15)
+		(end 147.15 71.65)
 		(width 0.2)
 		(layer "F.Cu")
-		(net "Net-(A1-GPIO0)")
+		(net "Net-(BT1--)")
 	)
 	(segment
-		(start 135.07 116.99)
-		(end 148.31 116.99)
+		(start 147.15 71.65)
+		(end 146.65 72.15)
 		(width 0.2)
 		(layer "F.Cu")
-		(net "Net-(A1-GPIO0)")
+		(net "Net-(BT1--)")
 	)
 	(segment
-		(start 153.85 111.45)
-		(end 153.85 75.21)
+		(start 147.09 68.09)
+		(end 147.15 68.15)
 		(width 0.2)
 		(layer "F.Cu")
-		(net "Net-(A1-GPIO0)")
+		(net "Net-(BT1--)")
 	)
 	(segment
-		(start 148.31 116.99)
-		(end 153.85 111.45)
+		(start 129.15 70.14)
+		(end 131.2 68.09)
 		(width 0.2)
 		(layer "F.Cu")
-		(net "Net-(A1-GPIO0)")
+		(net "Net-(BT1--)")
+	)
+	(segment
+		(start 131.2 68.09)
+		(end 147.09 68.09)
+		(width 0.2)
+		(layer "F.Cu")
+		(net "Net-(BT1--)")
+	)
+	(via
+		(at 146.65 72.15)
+		(size 0.6)
+		(drill 0.3)
+		(layers "F.Cu" "B.Cu")
+		(net "Net-(BT1--)")
+	)
+	(segment
+		(start 146.65 72.15)
+		(end 146.65 83.15)
+		(width 0.2)
+		(layer "B.Cu")
+		(net "Net-(BT1--)")
+	)
+	(segment
+		(start 138.65 86.15)
+		(end 141.15 88.65)
+		(width 0.2)
+		(layer "B.Cu")
+		(net "Net-(BT1--)")
+	)
+	(segment
+		(start 146.65 83.15)
+		(end 141.15 88.65)
+		(width 0.2)
+		(layer "B.Cu")
+		(net "Net-(BT1--)")
 	)
 	(segment
@@
 	)
 	(segment
+		(start 153.85 75.21)
+		(end 156.85 72.21)
+		(width 0.2)
+		(layer "F.Cu")
+		(net "Net-(A1-GPIO0)")
+	)
+	(segment
+		(start 135.07 116.99)
+		(end 148.31 116.99)
+		(width 0.2)
+		(layer "F.Cu")
+		(net "Net-(A1-GPIO0)")
+	)
+	(segment
+		(start 153.85 111.45)
+		(end 153.85 75.21)
+		(width 0.2)
+		(layer "F.Cu")
+		(net "Net-(A1-GPIO0)")
+	)
+	(segment
+		(start 148.31 116.99)
+		(end 153.85 111.45)
+		(width 0.2)
+		(layer "F.Cu")
+		(net "Net-(A1-GPIO0)")
+	)
+	(segment
 		(start 122.65 86.15)
 		(end 128.15 80.65)
@@
 		(net "Net-(A1-VSYS)")
 	)
-	(segment
-		(start 147.15 68.15)
-		(end 147.15 71.65)
-		(width 0.2)
-		(layer "F.Cu")
-		(net "Net-(BT1--)")
-	)
-	(segment
-		(start 147.15 71.65)
-		(end 146.65 72.15)
-		(width 0.2)
-		(layer "F.Cu")
-		(net "Net-(BT1--)")
-	)
-	(segment
-		(start 147.09 68.09)
-		(end 147.15 68.15)
-		(width 0.2)
-		(layer "F.Cu")
-		(net "Net-(BT1--)")
-	)
-	(segment
-		(start 129.15 70.14)
-		(end 131.2 68.09)
-		(width 0.2)
-		(layer "F.Cu")
-		(net "Net-(BT1--)")
-	)
-	(segment
-		(start 131.2 68.09)
-		(end 147.09 68.09)
-		(width 0.2)
-		(layer "F.Cu")
-		(net "Net-(BT1--)")
-	)
-	(via
-		(at 146.65 72.15)
-		(size 0.6)
-		(drill 0.3)
-		(layers "F.Cu" "B.Cu")
-		(net "Net-(BT1--)")
-	)
-	(segment
-		(start 146.65 72.15)
-		(end 146.65 83.15)
-		(width 0.2)
-		(layer "B.Cu")
-		(net "Net-(BT1--)")
-	)
-	(segment
-		(start 138.65 86.15)
-		(end 141.15 88.65)
-		(width 0.2)
-		(layer "B.Cu")
-		(net "Net-(BT1--)")
-	)
-	(segment
-		(start 146.65 83.15)
-		(end 141.15 88.65)
-		(width 0.2)
-		(layer "B.Cu")
-		(net "Net-(BT1--)")
-	)
-	(segment
-		(start 143.6125 110.65)
-		(end 143.6125 109.1875)
-		(width 0.2)
-		(layer "F.Cu")
-		(net "Net-(BT1-+)")
-	)
-	(segment
-		(start 143.6125 109.1875)
-		(end 144.15 108.65)
-		(width 0.2)
-		(layer "F.Cu")
-		(net "Net-(BT1-+)")
-	)
-	(via
-		(at 144.15 108.65)
-		(size 0.6)
-		(drill 0.3)
-		(layers "F.Cu" "B.Cu")
-		(net "Net-(BT1-+)")
-	)
-	(segment
-		(start 130.85 93.65)
-		(end 130.85 83.65)
-		(width 0.2)
-		(layer "B.Cu")
-		(net "Net-(BT1-+)")
-	)
-	(segment
-		(start 130.85 83.65)
-		(end 141.15 73.35)
-		(width 0.2)
-		(layer "B.Cu")
-		(net "Net-(BT1-+)")
-	)
-	(segment
-		(start 141.15 105.65)
-		(end 141.15 103.95)
-		(width 0.2)
-		(layer "B.Cu")
-		(net "Net-(BT1-+)")
-	)
-	(segment
-		(start 144.15 108.65)
-		(end 141.15 105.65)
-		(width 0.2)
-		(layer "B.Cu")
-		(net "Net-(BT1-+)")
-	)
-	(segment
-		(start 141.15 103.95)
-		(end 130.85 93.65)
-		(width 0.2)
-		(layer "B.Cu")
-		(net "Net-(BT1-+)")
-	)
 	(zone
