File: e.kicad_sch (KiCad schematic)
At the start: 10 parts, among them SW1 usr, SW2 rst, U1 Display_ST7789, U2 MAX98357A

Commit message: almost done i hope
Parts:
- removed R3: 10K, Resistor_SMD:R_1206_3216Metric, symbol Device:R_Small_US
Connections:
- net +3V0: now also BT1.1 (+)
Other:
- moved on the sheet: BT1, SW1
Changed lines of the file:
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@@
 	(text "THIS IS THE 1.54\" \nVERSION BTW\n<<<<<<<<<<"
 		(exclude_from_sim no)
-		(at 226.314 87.122 0)
+		(at 225.044 86.868 0)
 		(effects
 			(font
@@
 	(text "switched from 2032 to 2430 because of\nthe way the 2430 battery hold is designed, \nits lowkey impossible to wire it backwards, \neliminating the need for schottky diode.\n\nbrand: keystone"
 		(exclude_from_sim no)
-		(at 78.486 46.228 0)
+		(at 65.532 44.45 0)
 		(effects
 			(font
@@
 	)
 	(no_connect
-		(at 50.8 63.5)
+		(at 95.25 54.61)
 	)
 	(no_connect
@@
 	(wire
 		(pts
-			(xy 53.34 34.29) (xy 53.34 38.1)
-		)
-		(stroke
-			(width 0)
-			(type default)
-		)
-	)
-	(wire
-		(pts
 			(xy 195.58 80.01) (xy 191.77 80.01)
 		)
@@
 	(wire
 		(pts
-			(xy 53.34 43.18) (xy 53.34 45.72)
+			(xy 97.79 34.29) (xy 97.79 36.83)
 		)
 		(stroke
@@
 	(wire
 		(pts
-			(xy 55.88 63.5) (xy 55.88 64.77)
+			(xy 100.33 54.61) (xy 100.33 55.88)
 		)
 		(stroke
@@
 	(symbol
 		(lib_id "power:GND")
-		(at 55.88 64.77 0)
+		(at 100.33 55.88 0)
 		(unit 1)
 		(body_style 1)
@@
 		(fields_autoplaced yes)
 		(property "Reference" "#PWR06"
-			(at 55.88 71.12 0)
+			(at 100.33 62.23 0)
 			(hide yes)
 			(show_name no)
@@
 		)
 		(property "Value" "GND"
-			(at 55.88 69.85 0)
+			(at 100.33 60.96 0)
 			(show_name no)
 			(do_not_autoplace no)
@@
 		)
 		(property "Footprint" ""
-			(at 55.88 64.77 0)
+			(at 100.33 55.88 0)
 			(hide yes)
 			(show_name no)
@@
 		)
 		(property "Datasheet" ""
-			(at 55.88 64.77 0)
+			(at 100.33 55.88 0)
 			(hide yes)
 			(show_name no)
@@
 		)
 		(property "Description" "Power symbol creates a global label with name \"GND\" , ground"
-			(at 55.88 64.77 0)
+			(at 100.33 55.88 0)
 			(hide yes)
 			(show_name no)
@@
 	(symbol
 		(lib_id "Switch:SW_SPDT")
-		(at 53.34 58.42 270)
+		(at 97.79 49.53 270)
 		(unit 1)
 		(body_style 1)
@@
 		(dnp no)
 		(property "Reference" "SW1"
-			(at 58.42 57.1499 90)
+			(at 102.87 48.2599 90)
 			(show_name no)
 			(do_not_autoplace no)
@@
 		)
 		(property "Value" "usr"
-			(at 58.42 59.6899 90)
+			(at 102.87 50.7999 90)
 			(show_name no)
 			(do_not_autoplace no)
@@
 		)
 		(property "Footprint" "Button_Switch_THT:SW_Slide_SPDT_Straight_CK_OS102011MS2Q"
-			(at 53.34 58.42 0)
+			(at 97.79 49.53 0)
 			(hide yes)
 			(show_name no)
@@
 		)
 		(property "Datasheet" ""
-			(at 45.72 58.42 0)
+			(at 90.17 49.53 0)
 			(hide yes)
 			(show_name no)
@@
 		)
 		(property "Description" "Switch, single pole double throw"
-			(at 53.34 58.42 0)
+			(at 97.79 49.53 0)
 			(hide yes)
 			(show_name no)
@@
 				(path "/8ebdc5a5-d325-4a55-9117-5b5015586df6"
 					(reference "SW1")
-					(unit 1)
-				)
-			)
-		)
-	)
-	(symbol
-		(lib_id "Device:R_Small_US")
-		(at 53.34 40.64 0)
-		(mirror y)
-		(unit 1)
-		(body_style 1)
-		(exclude_from_sim no)
-		(in_bom yes)
-		(on_board yes)
-		(in_pos_files yes)
-		(dnp no)
-		(property "Reference" "R3"
-			(at 50.8 39.3699 0)
-			(show_name no)
-			(do_not_autoplace no)
-			(effects
-				(font
-					(size 1.27 1.27)
-				)
-				(justify left)
-			)
-		)
-		(property "Value" "10K"
-			(at 50.8 41.9099 0)
-			(show_name no)
-			(do_not_autoplace no)
-			(effects
-				(font
-					(size 1.27 1.27)
-				)
-				(justify left)
-			)
-		)
-		(property "Footprint" "Resistor_SMD:R_1206_3216Metric"
-			(at 53.34 40.64 0)
-			(hide yes)
-			(show_name no)
-			(do_not_autoplace no)
-			(effects
-				(font
-					(size 1.27 1.27)
-				)
-			)
-		)
-		(property "Datasheet" ""
-			(at 53.34 40.64 0)
-			(hide yes)
-			(show_name no)
-			(do_not_autoplace no)
-			(effects
-				(font
-					(size 1.27 1.27)
-				)
-			)
-		)
-		(property "Description" "Resistor, small US symbol"
-			(at 53.34 40.64 0)
-			(hide yes)
-			(show_name no)
-			(do_not_autoplace no)
-			(effects
-				(font
-					(size 1.27 1.27)
-				)
-			)
-		)
-		(pin "1"
-		)
-		(pin "2"
-		)
-		(instances
-			(project "e"
-				(path "/8ebdc5a5-d325-4a55-9117-5b5015586df6"
-					(reference "R3")
 					(unit 1)
 				)
@@
 	(symbol
 		(lib_id "power:+3V0")
-		(at 53.34 34.29 0)
+		(at 97.79 34.29 0)
 		(unit 1)
 		(body_style 1)
@@
 		(fields_autoplaced yes)
 		(property "Reference" "#PWR05"
-			(at 53.34 38.1 0)
+			(at 97.79 38.1 0)
 			(hide yes)
 			(show_name no)
@@
 		)
 		(property "Value" "+3V0"
-			(at 53.34 29.21 0)
+			(at 97.79 29.21 0)
 			(show_name no)
 			(do_not_autoplace no)
@@
 		)
 		(property "Footprint" ""
-			(at 53.34 34.29 0)
+			(at 97.79 34.29 0)
 			(hide yes)
 			(show_name no)
@@
 		)
 		(property "Datasheet" ""
-			(at 53.34 34.29 0)
+			(at 97.79 34.29 0)
 			(hide yes)
 			(show_name no)
@@
 		)
 		(property "Description" "Power symbol creates a global label with name \"+3V0\""
-			(at 53.34 34.29 0)
+			(at 97.79 34.29 0)
 			(hide yes)
 			(show_name no)
@@
 	(symbol
 		(lib_id "Device:Battery_Cell")
-		(at 53.34 50.8 0)
-		(mirror y)
+		(at 97.79 41.91 0)
 		(unit 1)
 		(body_style 1)
@@
 		(dnp no)
 		(property "Reference" "BT1"
-			(at 49.53 47.6884 0)
+			(at 101.6 38.7984 0)
 			(show_name no)
 			(do_not_autoplace no)
@@
 		)
 		(property "Value" "CR2430"
-			(at 49.53 50.2284 0)
+			(at 101.6 41.3384 0)
 			(show_name no)
 			(do_not_autoplace no)
@@
 		)
 		(property "Footprint" "Battery:BatteryHolder_Keystone_3008_1x2450"
-			(at 53.34 49.276 90)
+			(at 97.79 40.386 90)
 			(hide yes)
 			(show_name no)
@@
 		)
 		(property "Datasheet" ""
-			(at 53.34 49.276 90)
+			(at 97.79 40.386 90)
 			(hide yes)
 			(show_name no)
@@
 		)
 		(property "Description" "Single-cell battery"
-			(at 53.34 50.8 0)
+			(at 97.79 41.91 0)
 			(hide yes)
 			(show_name no)
@@
 		)
 		(property "Sim.Device" "V"
-			(at 53.34 50.8 0)
+			(at 97.79 41.91 0)
 			(hide yes)
 			(show_name no)
@@
 		)
 		(property "Sim.Type" "DC"
-			(at 53.34 50.8 0)
+			(at 97.79 41.91 0)
 			(hide yes)
 			(show_name no)
@@
 		)
 		(property "Sim.Pins" "1=+ 2=-"
-			(at 53.34 50.8 0)
-			(hide yes)
-			(show_name no)
+			(at 97.79 41.91 0)
+			(hide yes)
+			(show_name no)
